File: 8bit converter.kicad_pcb (KiCad board)
At the start: 2 copper layers, 125 x 90 mm, 36 parts, among them CN1 10220-55G3PC, J1 CONBNC002, SW2 TL1105SF160Q, U1 SN74LV1T34DBVR, U10 SC0915, U2 SN74LV1T34DBVR, U3 SN74LV1T34DBVR, U4 SN74LV1T34DBVR, U5 SN74LV1T34DBVR, U6 SN74LV1T34DBVR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

Commit message: PCB_edit
Parts:
- removed ${REFERENCE}: ${VALUE}, PcbObject:Logo
- removed C13, C14, C3, C4, C7, C8, C9: Value, Basic:CAP1005m
- removed PH1: PinHeader4x1, PinHeader:PinHeader4x1
- removed SW2: TL1105SF160Q, Switch:TL1105SF160Q
- added C19: 0.1uF, Basic:CAP1608m, F.Cu at (151.7, 46.3)
- added C20: 0.1uF, Basic:CAP1608m, F.Cu at (109.2, 99.3)
- added C21: 0.1uF, Basic:CAP1608m, F.Cu at (158.2, 46.3)
- added C22: 0.1uF, Basic:CAP1608m, F.Cu at (151.7, 58.3)
- added C23: 0.1uF, Basic:CAP1608m, F.Cu at (158.2, 58.3)
- added C24: 0.1uF, Basic:CAP1608m, F.Cu at (151.7, 70.3)
- added C25: 0.1uF, Basic:CAP1608m, F.Cu at (158.2, 70.3)
- added C26: 0.1uF, Basic:CAP1608m, F.Cu at (151.7, 82.3)
- added C27: 0.1uF, Basic:CAP1608m, F.Cu at (158.2, 82.3)
- added C28: 0.1uF, Basic:CAP1608m, F.Cu at (151.7, 94.3)
- added C29: 0.1uF, Basic:CAP1608m, F.Cu at (158.2, 94.3)
- added C30: 0.1uF, Basic:CAP1608m, F.Cu at (151.7, 106.3)
- added C31: 0.1uF, Basic:CAP1608m, F.Cu at (158.2, 106.3)
- added C32: 0.1uF, Basic:CAP1608m, F.Cu at (151.7, 118.3)
- added C33: 0.1uF, Basic:CAP1608m, F.Cu at (158.2, 118.3)
- added C34: 0.1uF, Basic:CAP1608m, F.Cu at (173.7, 120.3)
- added C35: 0.1uF, Basic:CAP1608m, F.Cu at (173.7, 113.8)
- added C36: 0.1uF, Basic:CAP1608m, F.Cu at (115.7, 99.3)
- added C37: 10uF, Basic:CAP1608m, F.Cu at (135.8, 87.5)
- added C38: 10uF, Basic:CAP1608m, F.Cu at (131.9, 87.5)
- added CN2: B4B-XH-A, Connector:B4B-XH-A, F.Cu at (215.6, 70.1)
- added D1: RB496EATR, Discrete:RB496EATR, F.Cu at (207.5, 45.0)
- added JP1: ~, Jumper:PAD_Short, F.Cu at (0.50, 0.60)
- added MH2: ~, PcbObject:HOLE_M3, F.Cu at (220.7, 130.3)
- added MH3: ~, PcbObject:HOLE_M3, F.Cu at (92.7, 44.3)
- added MH4: ~, PcbObject:HOLE_M3, F.Cu at (92.7, 130.3)
- added R10: 10k, Basic:REG1608m, F.Cu at (162.7, 111.3)
- added R11: 10k, Basic:REG1608m, F.Cu at (162.7, 123.3)
- added R12: 10k, Basic:REG1608m, F.Cu at (178.7, 109.3)
- added R13: 10k, Basic:REG1608m, F.Cu at (120.2, 104.3)
- added R3: 2.2k, Basic:REG1608m, F.Cu at (207.2, 68.8)
- added R4: 10k, Basic:REG1608m, F.Cu at (162.7, 75.3)
- added R5: 2.2k, Basic:REG1608m, F.Cu at (207.2, 63.9)
- added R6: 10k, Basic:REG1608m, F.Cu at (162.7, 63.3)
- added R7: 10k, Basic:REG1608m, F.Cu at (162.7, 87.3)
- added R8: 10k, Basic:REG1608m, F.Cu at (162.7, 51.3)
- added R9: 10k, Basic:REG1608m, F.Cu at (162.7, 99.3)
- added SW1: PN11SHNA03QE, Switch:PN11SHNA03QE, F.Cu at (202.7, 122.8)
- C1, C2: value Value -> 10uf; footprint Basic:CAP1005m -> Basic:CAP1608m
- R2: value Value -> 2.2k
- moved CN1 89.1 mm to (120.1, 49.3), turned to 180 degrees
- moved PS1 86.6 mm to (104.3, 68.1)
- moved J1 85.2 mm to (119.2, 124.8), turned to 0 degrees
- moved R2 84.6 mm to (204.2, 90.8), turned to 90 degrees
- moved MH1 80.0 mm to (220.7, 44.3)
- moved C1 68.9 mm to (108.7, 59.3)
- moved U10 67.1 mm to (188.9, 67.5)
- moved C2 56.7 mm to (108.7, 62.3)
- moved D10 43.0 mm to (109.2, 104.3), turned to 180 degrees
- moved U8 35.2 mm to (178.7, 113.8), turned to 90 degrees
- moved D9 31.8 mm to (178.7, 120.3), turned to -90 degrees
- moved U9 29.8 mm to (115.7, 104.3)
- moved U7 28.7 mm to (158.2, 123.3)
- moved D8 25.6 mm to (151.7, 123.3), turned to 180 degrees
- moved U6 23.2 mm to (158.2, 111.3)
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Connections:
- C1 pad 1: +5V -> GND
- C1 pad 2: GND -> /+12V
- C2 pad 1: +5V -> GND
- C2 pad 2: GND -> /+12V
- CN1 pad 1: /0_5V_MUX7 -> /o_5V_MUX7
- CN1 pad 11: /0_5V_MUX6 -> /o_5V_MUX6
- CN1 pad 12: /0_5V_MUX4 -> /o_5V_MUX4
- CN1 pad 13: /0_5V_MUX2 -> /o_5V_MUX2
- CN1 pad 14: /0_5V_MUX0 -> /o_5V_MUX0
- CN1 pad 2: /0_5V_MUX5 -> /o_5V_MUX5
- CN1 pad 3: /0_5V_MUX3 -> /o_5V_MUX3
- CN1 pad 4: /0_5V_MUX1 -> /o_5V_MUX1
- CN1 pad 7: unconnected-(CN1-Pad7) -> GND
- CN1 pad 9: unconnected-(CN1-Pad9) -> /+12V
- CN1 pad MH1: unconnected-(CN1-PadMH1) -> GND
- CN1 pad MH2: unconnected-(CN1-PadMH2) -> GND
- D10 pad 3: /o_TRIG -> /o_TRIG_BNC
- D2 pad 3: /o_MUX0 -> /o_5V_MUX0
- D3 pad 3: /o_MUX1 -> /o_5V_MUX1
- D4 pad 3: /o_MUX2 -> /o_5V_MUX2
- D5 pad 3: /o_MUX3 -> /o_5V_MUX3
- D6 pad 3: /o_MUX4 -> /o_5V_MUX4
- D7 pad 3: /o_MUX5 -> /o_5V_MUX5
- D8 pad 3: /o_MUX6 -> /o_5V_MUX6
- D9 pad 3: /o_MUX7 -> /o_5V_MUX7
- PS1 pad 1: unconnected-(PS1-RC-Pad1) -> Net-(PS1-RC)
- U1 pad 4: /0_5V_MUX0 -> /o_5V_MUX0
- U10 pad 11: /0_TRIG -> /o_TRIG
- U10 pad 14: /SDA -> unconnected-(U10-GP10(SPI1_SCK)-Pad14)
- U10 pad 15: /SCL -> unconnected-(U10-GP11(SPI1_TX)-Pad15)
- U10 pad 31: unconnected-(U10-GP26-Pad31) -> /SDA
- U10 pad 32: unconnected-(U10-GP27-Pad32) -> /SCL
- U10 pad 36: unconnected-(U10-3V3_OUT-Pad36) -> +3.3V
- U10 pad 39: unconnected-(U10-VSYS-Pad39) -> +5V
- U10 pad 40: +5V -> Net-(D1-A_2)
- U2 pad 4: /0_5V_MUX1 -> /o_5V_MUX1
- U3 pad 4: /0_5V_MUX2 -> /o_5V_MUX2
- U4 pad 4: /0_5V_MUX3 -> /o_5V_MUX3
- U5 pad 4: /0_5V_MUX4 -> /o_5V_MUX4
- U6 pad 4: /0_5V_MUX5 -> /o_5V_MUX5
- U7 pad 4: /0_5V_MUX6 -> /o_5V_MUX6
- U8 pad 4: /0_5V_MUX7 -> /o_5V_MUX7
Routing:
- net +5V: track 0.00 -> 167.0 mm, vias 0 -> 23
- net /o_5V_MUX7: track 0.00 -> 135.1 mm, vias 0 -> 1
- net GND: track 0.00 -> 122.2 mm, vias 0 -> 64
- net /o_5V_MUX6: track 0.00 -> 118.5 mm
- net /o_5V_MUX5: track 0.00 -> 101.6 mm
- net /o_5V_MUX4: track 0.00 -> 93.7 mm, vias 0 -> 1
- net /o_5V_MUX3: track 0.00 -> 87.7 mm
- net /o_5V_MUX2: track 0.00 -> 79.6 mm, vias 0 -> 1
- net /o_MUX6: track 0.00 -> 74.4 mm
- net /+12V: track 0.00 -> 74.0 mm
- net +3.3V: track 0.00 -> 72.4 mm
- net /o_MUX5: track 0.00 -> 67.9 mm
- net /o_MUX4: track 0.00 -> 60.5 mm
- net /o_5V_MUX1: track 0.00 -> 57.5 mm
- net /o_MUX7: track 0.00 -> 53.5 mm
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- added copper zone on In2.Cu, net +5V
- added copper zone on B.Cu, net GND
- added copper zone on F.Cu, net GND
- added copper zone on In1.Cu, net GND
Other:
- board size 125 x 90 mm -> 135 x 93 mm
- copper layers 2 -> 4

Commit message: PCB_check
Parts:
- added ${REFERENCE}: ${VALUE}, PcbObject:Logo_S, F.Cu at (112.2, 97.3)
- moved JP1 118.9 mm to (98.2, 68.3), turned to 90 degrees
- moved C20 28.5 mm to (137.7, 100.8), turned to 90 degrees
- moved D10 23.8 mm to (132.7, 100.8), turned to 90 degrees
- moved C36 23.4 mm to (137.7, 107.3), turned to 90 degrees
- moved U9 17.3 mm to (132.7, 107.3), turned to -90 degrees
- moved R13 14.6 mm to (132.7, 111.8), turned to 180 degrees
- moved D5 12.0 mm to (151.7, 87.3)
- moved D6 12.0 mm to (151.7, 99.3)
- moved U4 12.0 mm to (158.2, 87.3)
- moved U5 12.0 mm to (158.2, 99.3)
- moved R3 2.03 mm to (205.2, 68.8)
- moved R5 2.00 mm to (205.2, 63.8)
- moved MH1 1.41 mm to (219.7, 45.3)
- moved MH2 1.41 mm to (219.7, 129.3)
- moved MH3 1.41 mm to (93.7, 45.3)
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Connections:
- MH1 pad 1: unconnected-(MH1-Pad1) -> GND
- MH2 pad 1: unconnected-(MH2-Pad1) -> GND
- MH3 pad 1: unconnected-(MH3-Pad1) -> GND
- MH4 pad 1: unconnected-(MH4-Pad1) -> GND
Routing:
- net /o_TRIG: track 6.17 -> 131.3 mm
- net +3.3V: track 72.4 -> 27.4 mm, vias 0 -> 3
- net +5V: track 167.0 -> 181.5 mm, vias 23 -> 22
- net /o_5V_MUX3: track 87.7 -> 75.3 mm
- net /o_5V_MUX4: track 93.7 -> 105.7 mm
- net /o_TRIG_BNC: track 36.7 -> 41.4 mm
- net /SDA: track 19.4 -> 20.8 mm
- net Net-(PS1-RC): track 6.66 -> 5.73 mm, vias 1 -> 0
- net GND: vias 64 -> 116
- added copper zone on In2.Cu, net +3.3V
Other:
- outline, holes or cut-outs redrawn
- board text added: "JOB6073_2026JUN"
- board text added: "TRG_OUT"
