File: 8bit converter.kicad_pcb (KiCad board)
At the start: 4 copper layers, 135 x 93 mm, 65 parts, among them CN1 10220-55G3PC, CN2 B4B-XH-A, J1 CONBNC002, SW1 PN11SHNA03QE, U1 SN74LV1T34DBVR, U10 SC0915, U2 SN74LV1T34DBVR, U3 SN74LV1T34DBVR, U4 SN74LV1T34DBVR, U5 SN74LV1T34DBVR, U6 SN74LV1T34DBVR, U7 SN74LV1T34DBVR, U8 SN74LV1T34DBVR, U9 SN74LV1T34DBVR

Commit message: beforeaddingPower
Routing:
- net /+12V: track 73.6 -> 79.2 mm
Changed lines of the file:
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@@
 		(grid_origin 89.2 40.8)
 		(pcbplotparams
-			(layerselection 0x00000000_00000000_55555555_5755f5ff)
+			(layerselection 0x00000000_00000000_55555555_5755757f)
 			(plot_on_all_layers_selection 0x00000000_00000000_00000000_00000000)
 			(disableapertmacros no)
@@
 			(outputformat 1)
 			(mirror no)
-			(drillshape 1)
+			(drillshape 0)
 			(scaleselection 1)
-			(outputdirectory "")
+			(outputdirectory "./")
 		)
 	)
@@
 	(gr_line
 		(start 89.2 41.8)
-		(end 89.2 132.833539)
+		(end 89.2 132.8)
 		(stroke
 			(width 0.05)
-			(type default)
+			(type solid)
 		)
 		(layer "Edge.Cuts")
@@
 		(stroke
 			(width 0.05)
-			(type default)
+			(type solid)
 		)
 		(layer "Edge.Cuts")
 	)
 	(gr_arc
-		(start 90.199379 133.799866)
-		(mid 89.504305 133.51877)
-		(end 89.2 132.833539)
+		(start 90.199379 133.7993)
+		(mid 89.492745 133.50661)
+		(end 89.2 132.8)
 		(stroke
 			(width 0.05)
-			(type default)
+			(type solid)
 		)
 		(layer "Edge.Cuts")
@@
 	(gr_line
 		(start 90.200029 40.799999)
-		(end 223.197373 40.797391)
+		(end 223.197373 40.8)
 		(stroke
 			(width 0.05)
-			(type default)
+			(type solid)
 		)
 		(layer "Edge.Cuts")
@@
 	)
 	(gr_arc
-		(start 223.197373 40.797391)
-		(mid 223.90448 41.090284)
-		(end 224.197373 41.797391)
+		(start 223.200014 40.794803)
+		(mid 223.907266 41.089376)
+		(end 224.2 41.797391)
 		(stroke
 			(width 0.05)
@@
 		(layer "Edge.Cuts")
 	)
-	(gr_line
+	(gr_arc
 		(start 224.2 132.8)
-		(end 224.2 41.8)
+		(mid 223.907118 133.507096)
+		(end 223.200031 133.8)
 		(stroke
 			(width 0.05)
@@
 		(layer "Edge.Cuts")
 	)
-	(gr_arc
-		(start 224.200031 132.800027)
-		(mid 223.907138 133.507134)
-		(end 223.200031 133.800027)
+	(gr_line
+		(start 224.2 132.8)
+		(end 224.2 41.8)
 		(stroke
 			(width 0.05)
@@
 	)
 	(segment
+		(start 130.11 47.71)
+		(end 130.2 47.8)
+		(width 0.6)
+		(layer "F.Cu")
+		(net "/+12V")
+	)
+	(segment
 		(start 109.2 45.3)
 		(end 109.2 79.8)
@@
 	)
 	(segment
-		(start 130.2 49.8)
+		(start 130.2 47.8)
 		(end 130.2 44.8)
 		(width 0.6)
 		(layer "F.Cu")
+		(net "/+12V")
+	)
+	(segment
+		(start 130.2 49.8)
+		(end 130.2 47.8)
+		(width 0.6)
+		(layer "F.Cu")
+		(net "/+12V")
+	)
+	(segment
+		(start 124.59 47.71)
+		(end 130.11 47.71)
+		(width 0.6)
+		(layer "F.Cu")
