File: 8bit converter.kicad_sch (KiCad schematic)
At the start: 44 parts, among them CN1 10220-55G3PC, J1 CONBNC002, SW2 TL1105SF160Q, U1 SN74LV1T34DBVR, U10 SC0915, U2 SN74LV1T34DBVR, U3 SN74LV1T34DBVR, U4 SN74LV1T34DBVR, U5 SN74LV1T34DBVR, U6 SN74LV1T34DBVR, U7 SN74LV1T34DBVR, U8 SN74LV1T34DBVR, U9 SN74LV1T34DBVR

Commit message: circuit_check
Parts:
- removed C1, C10, C11, C12, C13, C14, C15, C16, C17, C18, C2, C3, C4, C5, C6, C7, C8, C9: Value, Basic:CAP1005m, symbol Basic:C1005m
- removed PH1: PinHeader4x1, PinHeader:PinHeader4x1, symbol PinHeader:PinHeader4x1
- added C19, C20, C21, C22, C23, C24, C25, C26, C27, C28, C29, C30, C31, C32, C33, C34, C35, C36: 0.1uF, Basic:CAP1608m, symbol Basic:C1608m
- added C37, C38: 10uF, Basic:CAP1608m, symbol Basic:C1608m
- added CN2: B4B-XH-A, Connector:B4B-XH-A, symbol Connector:B4B-XH-A
- added D1: RB496EATR, Discrete:RB496EATR, symbol Discrete:RB496EATR
- added JP1: (no value), Jumper:PAD_Short, symbol Jumper:PAD_Short
- added R10, R11, R12, R13, R4, R6, R7, R8, R9: 10k, Basic:REG1608m, symbol Basic:R1608m
- added R3, R5: 2.2k, Basic:REG1608m, symbol Basic:R1608m
Connections:
- net +12V: now also CN1.9
- net +3.3V: now also U10.36 (3V3_OUT), R3.2, R5.2
- net +5V: now also U10.39 (VSYS), C19.2, C20.2, C21.2, C22.1, C23.2, C24.2, C25.1, C26.1, C27.2, C28.1, C29.2, C30.1, C31.2, C32.1, C33.2, C34.1, C35.2, C36.1, C37.1, C38.1, CN2.3, D1.4 (K_2); no longer U10.40 (VBUS)
- net 0_5V_MUX0: now also D2.3
- net 0_5V_MUX1: now also D3.3
- net 0_5V_MUX2: now also D4.3
- net 0_5V_MUX3: now also D5.3
- net 0_5V_MUX4: now also D6.3
- net 0_5V_MUX5: now also D7.3
- net 0_5V_MUX6: now also D8.3
- net 0_5V_MUX7: now also D9.3
- net GND: now also CN1.7, CN1.MH1, CN1.MH2, C19.1, C20.1, C21.1, C22.2, C23.1, C24.1, C25.2, C26.2, C27.1, C28.2, C29.1, C30.2, C31.1, C32.2, C33.1, C34.2, C35.1, C36.2, C37.2, C38.2, CN2.4, JP1.1, R10.2, R11.2, R12.2, R13.2, R4.2, R6.2, R7.2, R8.2, R9.2
- net SCL: now also U10.32 (GP27), CN2.2, R5.1; no longer U10.15 (GP11(SPI1_TX))
- net SDA: now also U10.31 (GP26), CN2.1, R3.1; no longer U10.14 (GP10(SPI1_SCK))
- net o_MUX0: now also R8.1; no longer D2.3
- net o_MUX1: now also R6.1; no longer D3.3
- net o_MUX2: now also R4.1; no longer D4.3
- net o_MUX3: now also R7.1; no longer D5.3
- net o_MUX4: now also R9.1; no longer D6.3
- net o_MUX5: now also R10.1; no longer D7.3
- net o_MUX6: now also R11.1; no longer D8.3
- net o_MUX7: now also R12.1; no longer D9.3
- net o_TRIG: now also R13.1; no longer D10.3
- net o_TRIG_BNC: now also D10.3
- net at PS1.1 (RC): now also JP1.2
- new net: D1.3 (A_2), U10.40 (VBUS)
Other:
- moved on the sheet: D10, D2, D3, D4, D5, D6, D7, D8, D9

Commit message: PCB_edit
Parts:
- removed SW2: TL1105SF160Q, Switch:TL1105SF160Q, symbol Switch:TL1105SF160Q
- added C1, C2: 10uf, Basic:CAP1608m, symbol Basic:C1608m
- added MH2, MH3, MH4: (no value), PcbObject:HOLE_M3, symbol PcbObject:MountHole_M3
- added SW1: PN11SHNA03QE, Switch:PN11SHNA03QE, symbol Switch:PN11SHNA03QE
- R2: value Value -> 2.2k
Connections:
- net 0_TRIG is gone; now on net o_TRIG: U10.11 (GP8(I2C1_SDA))
- net +12V: now also C1.2, C2.2
- net GND: now also C1.1, C2.1, SW1.1 (NO)
- net at R2.1, U10.21 (GP16): now also SW1.2 (COM)
- net 0_5V_MUX0 renamed o_5V_MUX0
- net 0_5V_MUX1 renamed o_5V_MUX1
- net 0_5V_MUX2 renamed o_5V_MUX2
- net 0_5V_MUX3 renamed o_5V_MUX3
- net 0_5V_MUX4 renamed o_5V_MUX4
- net 0_5V_MUX5 renamed o_5V_MUX5
- net 0_5V_MUX6 renamed o_5V_MUX6
- net 0_5V_MUX7 renamed o_5V_MUX7
Other:
- moved on the sheet: C19, C20, C21, C22, C23, C24, C25, C26, C27, C28, C29, C30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

Commit message: PCB_check
Connections:
- net GND: now also MH1.1, MH2.1, MH3.1, MH4.1
